Commit message: mujoco motion controller tuning of the kinova arm done

File: docker/kortex_overrides/gen3_lite_kortex.ros2_control.xacro (robot description, xacro)
@@ -4,5 +4,5 @@
   kortex_description/arms/gen3_lite/6dof/urdf/kortex.ros2_control.xacro
   (vendor original, never edited directly — see mujoco_installation_sequence.md).
-  Diff from the vendor original, two changes only:
+  Diff from the vendor original, three changes:
     1. New `sim_mujoco` param + hardware-plugin branch, added following the exact
        same pattern already used here for sim_gazebo/sim_ignition/sim_isaac —
@@ -15,13 +15,32 @@
        runtime error: "Joint joint_1 needs a positive kp parameter for position
        fallback control" even with kp present but in the wrong XML location).
-       Required by MujocoRosSystem's fallback PD-control path (mujoco_ros_system.cpp,
-       reviewed during the mujoco_ros_pkgs integration) whenever a joint has no
-       matching named MuJoCo actuator ({joint}_act_pos) — which is our case,
-       since the scene doesn't hand-author actuators for these joints.
-  kp values below are UNTUNED STARTING POINTS, not measured/verified — same
-  placeholder status as OTHER_ARM_KEEPOUT in kinova_pick_planner.py. Expect to
-  adjust once the arm can actually be watched moving in MuJoCo: too low and it
-  won't track the commanded position with any authority, too high and it will
-  oscillate/overshoot.
+       Required whenever a joint has no matching named MuJoCo actuator
+       ({joint}_act_pos) — which is our case, since the scene doesn't hand-author
+       actuators for these joints. NOTE: despite "PD" naming conventions elsewhere,
+       this fallback (mujoco_ros_system.cpp, reviewed directly) is pure-P for the
+       position command interface: effort = kp * (cmd - actual), full stop — `kv`
+       exists in the same source but is only ever read for a *separate* velocity
+       command-interface fallback, never combined with kp here. Any damping/D-term
+       behavior has to come from the physics model itself (see the `damping`
+       attribute added to each <joint> in mujoco_scenes/gen3_lite.xml), not from
+       this controller.
+    3. Added an `effort_limit` param alongside `kp` on every actuated <joint>,
+       clamping the fallback's otherwise-unbounded P-control torque (defaults to
+       numeric_limits::max() if absent — confirmed by source review, not assumed).
+       Values are the real per-joint torque limits from the vendor URDF's own
+       <limit effort="..."/> tags (gen3_lite_macro.xacro for joints 1-6,
+       gen3_lite_2f_macro.xacro's 0/0.85-range variant for the gripper) — the same
+       numbers already present, inertly, as `actuatorfrcrange` in the converted
+       gen3_lite.xml (inert because that attribute only constrains MuJoCo
+       <actuator> elements, which this model doesn't define). Added *before*
+       raising kp values below, specifically so a higher kp can't demand
+       physically-unrealistic torque.
+  kp values below are UNTUNED STARTING POINTS, being tuned empirically via a
+  scripted step-response test (send a step goal through joint_trajectory_controller,
+  record /joint_states, measure overshoot/settle error) — see
+  mujoco_installation_sequence.md for the measured results and reasoning behind
+  each value. Too low and the joint can't hold position against gravity (measured:
+  joint_2 at kp=50 settled ~0.2 rad past a commanded target and stayed there —
+  gravity droop, not oscillation); too high and it will overshoot/oscillate.
   All joint limits (min/max) below are copied verbatim from the vendor original
   — not modified, not re-derived — these are the ones to trust as correct.
@@ -124,4 +143,5 @@
       <joint name="${prefix}joint_1">
         <param name="kp">50.0</param>
+        <param name="effort_limit">10.0</param>
         <command_interface name="position">
           <param name="min">-2.69</param>
@@ -135,5 +155,6 @@
       </joint>
       <joint name="${prefix}joint_2">
-        <param name="kp">50.0</param>
+        <param name="kp">250.0</param>
+        <param name="effort_limit">14.0</param>
         <command_interface name="position">
           <param name="min">-2.69</param>
@@ -148,4 +169,5 @@
       <joint name="${prefix}joint_3">
         <param name="kp">50.0</param>
+        <param name="effort_limit">10.0</param>
         <command_interface name="position">
           <param name="min">-2.69</param>
@@ -160,4 +182,5 @@
       <joint name="${prefix}joint_4">
         <param name="kp">30.0</param>
+        <param name="effort_limit">7.0</param>
         <command_interface name="position">
           <param name="min">-2.59</param>
@@ -172,4 +195,5 @@
       <joint name="${prefix}joint_5">
         <param name="kp">30.0</param>
+        <param name="effort_limit">7.0</param>
         <command_interface name="position">
           <param name="min">-2.57</param>
@@ -184,4 +208,5 @@
       <joint name="${prefix}joint_6">
         <param name="kp">30.0</param>
+        <param name="effort_limit">7.0</param>
         <command_interface name="position">
           <param name="min">-2.59</param>
@@ -198,4 +223,5 @@
           <joint name="${prefix}right_finger_bottom_joint">
             <param name="kp">10.0</param>
+            <param name="effort_limit">50.0</param>
             <command_interface name="position"/>
             <state_interface name="position"/>
@@ -207,4 +233,5 @@
         <joint name="${prefix}right_finger_bottom_joint">
           <param name="kp">10.0</param>
+          <param name="effort_limit">50.0</param>
           <command_interface name="position"/>
           <state_interface name="position"/>

Commit message: mujoco arm A execute:  pick cup done

File: docker/kortex_overrides/gen3_lite_kortex.ros2_control.xacro (robot description, xacro)
@@ -222,5 +222,5 @@
         <xacro:unless value="${moveit_active}">
           <joint name="${prefix}right_finger_bottom_joint">
-            <param name="kp">10.0</param>
+            <param name="kp">50.0</param>
             <param name="effort_limit">50.0</param>
             <command_interface name="position"/>
@@ -232,5 +232,5 @@
       <xacro:if value="${moveit_active}">
         <joint name="${prefix}right_finger_bottom_joint">
-          <param name="kp">10.0</param>
+          <param name="kp">50.0</param>
           <param name="effort_limit">50.0</param>
           <command_interface name="position"/>

File: docker/kortex_overrides/gen3_lite_macro.xacro (robot description, xacro)
@@ -8,11 +8,22 @@
     1. `sim_mujoco:=false` added to the macro's param list.
     2. A new `xacro:if value="${sim_mujoco}"` block setting ros2_control_name to
-       "MujocoRosSystem" (the other branches here set it per-backend too, e.g.
-       "GenericSystem" for fake hardware — this is just a label passed to
-       <ros2_control name="...">, not the actual plugin class, which is chosen
-       separately in kortex.ros2_control.xacro).
+       "${prefix}MujocoRosSystem" (the other branches here set it per-backend
+       too, e.g. "GenericSystem" for fake hardware — this is just a label
+       passed to <ros2_control name="...">, not the actual plugin class, which
+       is chosen separately in kortex.ros2_control.xacro).
     3. `sim_mujoco` added to the exclusion list on the real-hardware `unless`
        block, and `sim_mujoco="${sim_mujoco}"` added to the xacro:kortex_ros2_control
        forwarding call.
+  Bug found and fixed during dual-arm work (see mujoco_motion_controller_tuning.md):
+  this branch originally set ros2_control_name to the bare literal
+  "MujocoRosSystem", NOT prefixed like the real-hardware branch a few lines down
+  (`${prefix}KortexMultiInterfaceHardware`). Harmless for a single arm, but with
+  two arms in one combined URDF both got the identical <ros2_control name=...>,
+  and mujoco_ros_control.cpp's resource_manager_->set_component_state(i.name, ...)
+  looks components up by that name — so the second arm's hardware component was
+  imported but silently never activated (symptom: its joint_trajectory_controller
+  failed to activate with "Not available" command interfaces, even though the
+  interfaces existed in the resource manager's inventory). Fixed by prefixing it,
+  matching the pattern already used one branch down.
   Everything else — all link/joint geometry, masses, inertias, mesh references,
   joint limits — is copied verbatim from the vendor original. Not modified, not
@@ -65,5 +76,5 @@
     <xacro:if value="${sim_mujoco}">
       <xacro:unless value="${moveit_active}">
-        <xacro:property name="ros2_control_name" value="MujocoRosSystem"/>
+        <xacro:property name="ros2_control_name" value="${prefix}MujocoRosSystem"/>
       </xacro:unless>
     </xacro:if>
